Commit message: Update urdf definition from rx90 manual

File: staubli/html/urdf/staubli_tx90_support/urdf/tx90-rx.urdf (robot description, URDF)
Before this commit: robot staubli_tx90, 10 links, 9 joints
Joints:
- joint base_link-base: origin xyz=0 0 0.478 rpy=0 0 0 -> xyz=0 0 0.420 rpy=0 0 0
- joint joint_1: origin xyz=0 0 0.478 rpy=0 0 0 -> xyz=0 0 0.420 rpy=0 0 0
- joint joint_2: origin xyz=0.050 0 0 rpy=0 0 0 -> xyz=0 0 0 rpy=0 0 0
- joint joint_3: origin xyz=0 0.05 0.425 rpy=0 0 0 -> xyz=0 0.0 0.450 rpy=0 0 0
- joint joint_5: origin xyz=0 0 0.425 rpy=0 0 0 -> xyz=0 0 0.450 rpy=0 0 0
- joint joint_6: origin xyz=0 0 0.100 rpy=0 0 0 -> xyz=0 0 0.085 rpy=0 0 0
