Commit message: Switch from ROS urdf to custom one

File: staubli/html/urdf/staubli_rx90/StaubliRX90.urdf (robot description, URDF)
Before this commit: robot staubli_tx90l, 10 links, 9 joints
Links:
- link base_link: geometry collision mesh filename=package://staubli_rx90/StaubliRX90-Base.stl scale=0.001 0.001 0.001; visual mesh filename=package://staubli_rx90/StaubliRX90-Base.stl scale=0.001 0.001 0.001
- link link_1: geometry collision mesh filename=package://staubli_rx90/StaubliRX90-Shoulder.stl scale=0.001 0.001 0.001; visual mesh filename=package://staubli_rx90/StaubliRX90-Shoulder.stl scale=0.001 0.001 0.001
- link link_2: mass 14.350897 -> 12.98711; geometry collision mesh filename=package://staubli_rx90/StaubliRX90-Arm.stl scale=0.001 0.001 0.001; visual mesh filename=package://staubli_rx90/StaubliRX90-Arm.stl scale=0.001 0.001 0.001
- link link_3: mass 7.501506 -> 7.50151; geometry collision mesh filename=package://staubli_rx90/StaubliRX90-Elbow.stl scale=0.001 0.001 0.001; visual mesh filename=package://staubli_rx90/StaubliRX90-Elbow.stl scale=0.001 0.001 0.001
- link link_4: mass 6.420429 -> 4.54015; geometry collision mesh filename=package://staubli_rx90/StaubliRX90-Forearm.stl scale=0.001 0.001 0.001; visual mesh filename=package://staubli_rx90/StaubliRX90-Forearm.stl scale=0.001 0.001 0.001
- link link_5: mass 0.568760 -> 0.56876; geometry collision mesh filename=package://staubli_rx90/StaubliRX90-Wrist.stl scale=0.001 0.001 0.001; visual mesh filename=package://staubli_rx90/StaubliRX90-Wrist.stl scale=0.001 0.001 0.001
- link link_6: mass 0.030977 -> 0.03098; geometry collision mesh filename=package://staubli_rx90/StaubliRX90-Flange.stl scale=0.001 0.001 0.001; visual mesh filename=package://staubli_rx90/StaubliRX90-Flange.stl scale=0.001 0.001 0.001
Joints:
- joint base_link-base: origin xyz=0 0 0.478 rpy=0 0 0 -> xyz=0 0 0.420 rpy=0 0 0
- joint joint_1: origin xyz=0 0 0.478 rpy=0 0 0 -> xyz=0 0 0.420 rpy=0 0 0
- joint joint_2: limit lower=-2.2689280275926285 upper=2.5743606466916362 effort=130.0 velocity=6.806784082777885 -> lower=-2.2689280275926285 upper=2.5743606466916362 effort=166.0 velocity=6.981317007977318; origin xyz=0.050 0 0 rpy=0 0 0 -> xyz=0 0 0 rpy=0 0 0
- joint joint_3: limit lower=-2.530727415391778 upper=2.530727415391778 effort=65.0 velocity=7.3303828583761845 -> lower=-2.530727415391778 upper=2.530727415391778 effort=76.0 velocity=7.504915783575617; origin xyz=0 0.05 0.500 rpy=0 0 0 -> xyz=0 0.0 0.450 rpy=0 0 0
- joint joint_5: origin xyz=0 0 0.550 rpy=0 0 0 -> xyz=0 0 0.450 rpy=0 0 0
- joint joint_6: origin xyz=0 0 0.100 rpy=0 0 0 -> xyz=0 0 0.085 rpy=0 0 0
